File: li-ion_BMS_PCB/BMS_IC_Circuit.kicad_sch (KiCad schematic)
At the start: 49 parts, among them J6 Conn_01x02, J7 Conn_01x02, J8 Conn_01x02

Commit message: progress
Parts:
- removed C17: 100n, Capacitor_SMD:C_0603_1608Metric, symbol Device:C
- removed J6: Conn_01x02, Connector_Wire:SolderWire-0.1sqmm_1x02_P3.6mm_D0.4mm_OD1mm, symbol Connector_Generic:Conn_01x02
- removed J7: Conn_01x02, Jumper:SolderJumper-2_P1.3mm_Open_Pad1.0x1.5mm, symbol Connector_Generic:Conn_01x02
- removed R15, R16: 10k, Resistor_SMD:R_0402_1005Metric, symbol Device:R
- removed TP1: TestPoint, TestPoint:TestPoint_Pad_D1.0mm, symbol Connector:TestPoint
- added J9: Conn_01x09, Connector_PinHeader_2.54mm:PinHeader_1x09_P2.54mm_Vertical, symbol Connector_Generic:Conn_01x09
- added JP1, JP2: SolderJumper_3_Open, Jumper:SolderJumper-3_P1.3mm_Open_Pad1.0x1.5mm_NumberLabels, symbol Jumper:SolderJumper_3_Open
- D1, D2: footprint (none) -> li-ion_BMS:SS34; LCSC (none) -> C8678
- J8: footprint Connector_Wire:SolderWire-0.1sqmm_1x02_P3.6mm_D0.4mm_OD1mm -> Connector_JST:JST_GH_SM02B-GHS-TB_1x02-1MP_P1.25mm_Horizontal; LCSC (none) -> C189893; now in the parts list
- R17: now fitted; now in the parts list
Connections:
- net FAULTN: now also J9.4 (Pin_4)
- net FAULTN_SAFE: now also J9.5 (Pin_5)
- net GND: now also J9.9 (Pin_9)
- net NSHIP: now also J9.3 (Pin_3)
- net RDY: now also J9.8 (Pin_8)
- net SCL: now also JP1.1 (A); no longer R2.2, U1.5 (SCL)
- net SDA: now also JP2.3 (B); no longer R1.2, U1.6 (SDA)
- net VREG_3V3: now also J9.1 (Pin_1)
- net WAKEUP: now also J9.2 (Pin_2)
- net at R18.1, R19.2: now also J8.1 (Pin_1); no longer J8.2 (Pin_2)
- net at U1.10 (OD): now also J8.2 (Pin_2); no longer J8.1 (Pin_1)
- new net: JP1.2 (C), R2.2, U1.5 (SCL)
- new net: JP2.2 (C), R1.2, U1.6 (SDA)
- new net SCL_EXT: J9.6 (Pin_6), JP1.3 (B)
- new net SDA_EXT: J9.7 (Pin_7), JP2.1 (A)
Other:
- note added: "Connector to external Nucleo-G071RB"
- note added: "Notes 1) The FUSE circuit is not present as I would like to save space on this version of the BMS. Refer to the STEVAL-L99615C circuit if implementation is needed 2) J8 can be connected to an NTC for temperature sensing. Enable by programming NTC_EN"
- note removed: "Notes 1) The FUSE circuit is not present as I would like to save space on this version of the BMS. Refer to the STEVAL-L99615C circuit if implementation is needed 2) Option to solder a push button to J6, allowing wakeup without using MCU 3) J7 can be solder bridged to ensure that the BMS is turned on in standby mode. 4) J8 can be soldered to an NTC for temperature sensing. Enable by programming N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"
- moved on the sheet: C16, D2
