File: li-ion_BMS_PCB/Battery_Interfacing_Circuit.kicad_sch (KiCad schematic)
At the start: 14 parts, among them J1 Conn_01x06_Pin, J2 Conn_Solder_Pad, J3 Conn_Solder_Pad, J4 Conn_Solder_Pad, J5 Conn_Solder_Pad, Q1 NMOS, Q2 NMOS

Commit message: progress
Parts:
- removed J1: Conn_01x06_Pin, Connector_JST:JST_GH_SM06B-GHS-TB_1x06-1MP_P1.25mm_Horizontal, symbol Connector:Conn_01x06_Pin
- removed TP10, TP11, TP8, TP9: TestPoint, TestPoint:TestPoint_Pad_D1.0mm, symbol Connector:TestPoint
- added J1: Conn_01x06, Connector_JST:JST_GH_SM06B-GHS-TB_1x06-1MP_P1.25mm_Horizontal, symbol Connector_Generic:Conn_01x06
- Q1: footprint (none) -> li-ion_BMS:JLCPCB-DFN-8(4.9x5.8); LCSC (none) -> C78118
- Q2: LCSC (none) -> C78118
Connections:
- net C0: now also J1.6 (Pin_6)
- net C1: now also J1.5 (Pin_5)
- net C2: now also J1.4 (Pin_4)
- net C3: now also J1.3 (Pin_3)
- net C4: now also J1.2 (Pin_2)
- net C5: now also J1.1 (Pin_1)
