File: li-ion_BMS_PCB/li-ion_BMS_PCB.kicad_sch (KiCad schematic)
At the start: 0 parts

Commit message: progress
Other:
- sheet BMS_IC_Circuit ports: added FAULTN, FAULTN_SAFE, NSHIP, RDY, VREG_3V3, WAKEUP; removed none
- sheet Battery_Interfacing_Circuit: file /home/sharkbonebroth/li-ion_BMS/li-ion_BMS_PCB/Battery_Interfacing_Circuit.kicad_sch -> Battery_Interfacing_Circuit.kicad_sch
- sheet MCU_Circuit ports: added FAULTN, FAULTN_SAFE, NSHIP, RDY, SCL, SDA, VREG_3V3, WAKEUP; removed none
Changed lines of the file:
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@@
+	(wire
+		(pts
+			(xy 78.74 105.41) (xy 87.63 105.41)
+		)
+		(stroke
+			(width 0)
+			(type default)
+		)
+	)
+	(wire
+		(pts
+			(xy 78.74 97.79) (xy 87.63 97.79)
+		)
+		(stroke
+			(width 0)
+			(type default)
+		)
+	)
+	(wire
+		(pts
+			(xy 78.74 95.25) (xy 87.63 95.25)
+		)
+		(stroke
+			(width 0)
+			(type default)
+		)
+	)
 	(wire
 		(pts
@@
 	(wire
 		(pts
+			(xy 78.74 90.17) (xy 87.63 90.17)
+		)
+		(stroke
+			(width 0)
+			(type default)
+		)
+	)
+	(wire
+		(pts
 			(xy 78.74 45.72) (xy 87.63 45.72)
 		)
@@
 	(wire
 		(pts
+			(xy 78.74 102.87) (xy 87.63 102.87)
+		)
+		(stroke
+			(width 0)
+			(type default)
+		)
+	)
+	(wire
+		(pts
+			(xy 78.74 100.33) (xy 87.63 100.33)
+		)
+		(stroke
+			(width 0)
+			(type default)
+		)
+	)
+	(wire
+		(pts
 			(xy 78.74 43.18) (xy 87.63 43.18)
 		)
@@
 	(wire
 		(pts
+			(xy 78.74 92.71) (xy 87.63 92.71)
+		)
+		(stroke
+			(width 0)
+			(type default)
+		)
+	)
+	(wire
+		(pts
 			(xy 78.74 71.12) (xy 87.63 71.12)
+		)
+		(stroke
+			(width 0)
+			(type default)
+		)
+	)
+	(wire
+		(pts
+			(xy 78.74 107.95) (xy 87.63 107.95)
 		)
 		(stroke
@@
 		)
 		(pin "SDA" input
-			(at 78.74 102.87 0)
+			(at 78.74 95.25 0)
 			(effects
 				(font
@@
 		)
 		(pin "SCL" input
-			(at 78.74 100.33 0)
+			(at 78.74 92.71 0)
 			(effects
 				(font
@@
 		(pin "VSC" input
 			(at 78.74 73.66 0)
+			(effects
+				(font
+					(size 1.27 1.27)
+				)
+				(justify right)
+			)
+		)
+		(pin "FAULTN_SAFE" input
+			(at 78.74 97.79 0)
+			(effects
+				(font
+					(size 1.27 1.27)
+				)
+				(justify right)
+			)
+		)
+		(pin "FAULTN" input
+			(at 78.74 100.33 0)
+			(effects
+				(font
+					(size 1.27 1.27)
+				)
+				(justify right)
+			)
+		)
+		(pin "RDY" input
+			(at 78.74 102.87 0)
+			(effects
+				(font
+					(size 1.27 1.27)
+				)
+				(justify right)
+			)
+		)
+		(pin "WAKEUP" input
+			(at 78.74 105.41 0)
+			(effects
+				(font
+					(size 1.27 1.27)
+				)
+				(justify right)
+			)
+		)
+		(pin "NSHIP" input
+			(at 78.74 107.95 0)
+			(effects
+				(font
+					(size 1.27 1.27)
+				)
+				(justify right)
+			)
+		)
+		(pin "VREG_3V3" input
+			(at 78.74 90.17 0)
 			(effects
 				(font
@@
 	)
 	(sheet
-		(at 87.63 92.71)
-		(size 43.18 17.78)
+		(at 87.63 87.63)
+		(size 43.18 22.86)
 		(fields_autoplaced yes)
 		(stroke
@@
 		)
 		(property "Sheetname" "MCU_Circuit"
-			(at 87.63 91.9984 0)
+			(at 87.63 86.9184 0)
 			(effects
 				(font
@@
 				)
 				(justify left top)
+			)
+		)
+		(pin "SCL" input
+			(at 87.63 92.71 180)
+			(effects
+				(font
+					(size 1.27 1.27)
+				)
+				(justify left)
+			)
+		)
+		(pin "NSHIP" input
+			(at 87.63 107.95 180)
+			(effects
+				(font
+					(size 1.27 1.27)
+				)
+				(justify left)
+			)
+		)
+		(pin "FAULTN_SAFE" input
+			(at 87.63 97.79 180)
+			(effects
+				(font
+					(size 1.27 1.27)
+				)
+				(justify left)
+			)
+		)
+		(pin "SDA" input
+			(at 87.63 95.25 180)
+			(effects
+				(font
+					(size 1.27 1.27)
+				)
+				(justify left)
+			)
+		)
+		(pin "RDY" input
+			(at 87.63 102.87 180)
+			(effects
+				(font
+					(size 1.27 1.27)
+				)
+				(justify left)
+			)
+		)
+		(pin "FAULTN" input
+			(at 87.63 100.33 180)
+			(effects
+				(font
+					(size 1.27 1.27)
+				)
+				(justify left)
+			)
+		)
+		(pin "WAKEUP" input
+			(at 87.63 105.41 180)
+			(effects
+				(font
+					(size 1.27 1.27)
+				)
+				(justify left)
+			)
+		)
+		(pin "VREG_3V3" input
+			(at 87.63 90.17 180)
+			(effects
+				(font
+					(size 1.27 1.27)
+				)
+				(justify left)
 			)
 		)
@@
 			)
 		)
-		(property "Sheetfile" "/home/sharkbonebroth/li-ion_BMS/li-ion_BMS_PCB/Battery_Interfacing_Circuit.kicad_sch"
+		(property "Sheetfile" "Battery_Interfacing_Circuit.kicad_sch"
 			(at 87.63 76.7846 0)
 			(effects
