File: li-ion_BMS_PCB/MCU_Circuit.kicad_sch (KiCad schematic)
At the start: 0 parts

Commit message: progress
Parts:
- added C19, C20: 15p, Capacitor_SMD:C_0603_1608Metric, symbol Device:C
- added C21, C23, C25: 100n, Capacitor_SMD:C_0402_1005Metric, symbol Device:C
- added C22, C24: 4.7u, Capacitor_SMD:C_0603_1608Metric, symbol Device:C
- added J10: Conn_01x07, Connector_PinHeader_2.54mm:PinHeader_1x07_P2.54mm_Vertical, symbol Connector_Generic:Conn_01x07
- added J11: Conn_01x04, Connector_JST:JST_GH_SM04B-GHS-TB_1x04-1MP_P1.25mm_Horizontal, symbol Connector_Generic:Conn_01x04
- added J6, J7: Conn_01x02, Connector_JST:JST_GH_SM02B-GHS-TB_1x02-1MP_P1.25mm_Horizontal, symbol Connector_Generic:Conn_01x02
- added R20, R24: 33k, Resistor_SMD:R_0402_1005Metric, symbol Device:R
- added U2: STM32G071RBTx, Package_QFP:LQFP-64_10x10mm_P0.5mm, symbol MCU_ST_STM32G0:STM32G071RBTx
- added Y1: 12.5p, li-ion_BMS:NX3215SA-32.768K-STD-MUA-8, symbol Device:Crystal
Connections:
- new net: J6.1 (Pin_1), R20.2, U2.55 (PD5)
- new net: C19.1, U2.4 (PC14), Y1.2
- new net: C20.1, U2.5 (PC15), Y1.1
- new net FAULTN: U2.23 (PA6)
- new net FAULTN_SAFE: U2.24 (PA7)
- new net GND: C19.2, C20.2, C21.2, C22.2, C23.2, C24.2, C25.2, J10.7 (Pin_7), J11.4 (Pin_4), J7.2 (Pin_2), R20.1, R24.1, U2.9 (VSS)
- new net MCO: J10.4 (Pin_4), U2.10 (PF0)
- new net NRST: C25.1, J10.1 (Pin_1), J7.1 (Pin_1), U2.12 (PF2)
- new net NSHIP: U2.63 (PB9)
- new net RDY: U2.27 (PB0)
- new net SCL: U2.33 (PB13)
- new net SCL_HOST: J11.1 (Pin_1), U2.37 (PA9/UCPD1_DBCC1)
- new net SDA: U2.34 (PB14)
- new net SDA_HOST: J11.2 (Pin_2), U2.42 (PA10/UCPD1_DBCC2)
- new net TCK: J10.2 (Pin_2), U2.46 (PA14)
- new net TMS: J10.3 (Pin_3), U2.45 (PA13)
- new net UART2_RX: J10.6 (Pin_6), U2.20 (PA3)
- new net UART2_TX: J10.5 (Pin_5), U2.19 (PA2)
- new net VREG_3V3: C21.1, C22.1, C23.1, C24.1, J6.2 (Pin_2), U2.6 (VBAT), U2.8 (VDD)
- new net WAKE: J11.3 (Pin_3), R24.2, U2.43 (PA11/PA9)
- new net WAKEUP: U2.22 (PA5)
- no-connect marks 0 -> 42
Other:
- note added: "Battery Check Button"
- note added: "MCU RESET Button"
- note added: "Notes 1) While the L9961 IC has a 3.3V LDO output for powering peripherals, it is only capable of sinking a maximum of 35mA (15mA during standby mode) 2) IC choice: STM32G071RB a) Exact same MCU that is used to interface with the STEVAL-L99615C, allowing us to reuse the sample test code provided without the corresponding Nucleo-G071RB board. b) Standby current consumption: ~0.5uA (RTC disabled), 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"
- note added: "STM32G071RB MCU Circuit"
- note added: "To External Host"
- note added: "To STLink"
- note removed: "Notes 1) While the L9961 IC has a 3.3V LDO output for powering peripherals, it is only capable of sinking a maximum of 35mA, which is insufficient since we want to be able to power LED indicators"
- note removed: "STM32F103C8T6 MCU Circuit"

Commit message: finished initial V1
Parts:
- added D10, D3, D4, D5, D6, D7, D8, D9: LED, LED_SMD:LED_0603_1608Metric, symbol Device:LED
- added R15, R22, R25, R27: 4.7k, Resistor_SMD:R_0402_1005Metric, symbol Device:R
- added R16: 33k, Resistor_SMD:R_0402_1005Metric, symbol Device:R
- added R21, R23, R26: 3.3k, Resistor_SMD:R_0402_1005Metric, symbol Device:R
- R20: value 33k -> 3.3k; LCSC C25779 -> C25890
Connections:
- net GND: now also D10.1 (K), D3.1 (K), D4.1 (K), D5.1 (K), D6.1 (K), D7.1 (K), D8.1 (K), D9.1 (K), R16.1; no longer R20.1
- net LEDWhite1: now reaches R20.2, U2.55 (PD5)
- net LEDWhite1: no longer J6.1 (Pin_1)
- net at U2.54 (PD4): now also J6.1 (Pin_1), R16.2
- net LEDRed1: now reaches U2.56 (PD6)
- net LEDRed1: now also R15.2
- net LEDWhite2: now reaches U2.57 (PB3)
- net LEDWhite2: now also R21.2
- net LEDRed2: now reaches U2.58 (PB4)
- net LEDRed2: now also R22.2
- net LEDWhite3: now reaches U2.59 (PB5)
- net LEDWhite3: now also R23.2
- net LEDRed3: now reaches U2.60 (PB6)
- net LEDRed3: now also R25.2
- net LEDWhite4: now reaches U2.61 (PB7)
- net LEDWhite4: now also R26.2
- net LEDRed4: now reaches U2.62 (PB8)
- net LEDRed4: now also R27.2
- new net: D6.2 (A), R22.1
- new net: D4.2 (A), R15.1
- new net: D3.2 (A), R20.1
- new net: D7.2 (A), R23.1
- new net: D5.2 (A), R21.1
- new net: D10.2 (A), R27.1
- new net: D8.2 (A), R25.1
- new net: D9.2 (A), R26.1
- no-connect marks 42 -> 34
Other:
- moved on the sheet: J10
