File: li-ion_BMS_PCB/li-ion_BMS_PCB.kicad_pcb (KiCad board)
At the start: 4 copper layers, 32 x 60 mm, 71 parts, among them J1 Conn_01x06, J10 Conn_01x07, J11 Conn_01x04, J2 Conn_Solder_Pad, J3 Conn_Solder_Pad, J4 Conn_Solder_Pad, J5 Conn_Solder_Pad, J6 Conn_01x02, J7 Conn_01x02, J8 Conn_01x02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

Commit message: finished initial V1
Parts:
- added D10: LED, LED_SMD:LED_0603_1608Metric, F.Cu at (134.3, 77.0)
- added D3: LED, LED_SMD:LED_0603_1608Metric, F.Cu at (117.7, 77.0)
- added D4: LED, LED_SMD:LED_0603_1608Metric, F.Cu at (119.3, 77.0)
- added D5: LED, LED_SMD:LED_0603_1608Metric, F.Cu at (122.7, 77.0)
- added D6: LED, LED_SMD:LED_0603_1608Metric, F.Cu at (124.3, 77.0)
- added D7: LED, LED_SMD:LED_0603_1608Metric, F.Cu at (127.7, 77.0)
- added D8: LED, LED_SMD:LED_0603_1608Metric, F.Cu at (129.3, 77.0)
- added D9: LED, LED_SMD:LED_0603_1608Metric, F.Cu at (132.7, 77.0)
- added R15: 4.7k, Resistor_SMD:R_0402_1005Metric, F.Cu at (119.3, 74.5)
- added R16: 33k, Resistor_SMD:R_0402_1005Metric, F.Cu at (121.5, 70.0)
- added R21: 3.3k, Resistor_SMD:R_0402_1005Metric, F.Cu at (122.7, 74.5)
- added R22: 4.7k, Resistor_SMD:R_0402_1005Metric, F.Cu at (124.3, 74.5)
- added R23: 3.3k, Resistor_SMD:R_0402_1005Metric, F.Cu at (127.7, 74.5)
- added R25: 4.7k, Resistor_SMD:R_0402_1005Metric, F.Cu at (129.3, 74.5)
- added R26: 3.3k, Resistor_SMD:R_0402_1005Metric, F.Cu at (132.7, 74.5)
- added R27: 4.7k, Resistor_SMD:R_0402_1005Metric, F.Cu at (134.3, 74.5)
- R20: value 33k -> 3.3k
- moved R20 7.38 mm to (117.7, 74.5), turned to 90 degrees
Connections:
- R20 pad 1: GND -> Net-(D3-A)
- R20 pad 2: Net-(J6-Pin_1) -> /MCU_Circuit/LEDWhite1
- U2 pad 54: unconnected-(U2-PD4-Pad54) -> Net-(J6-Pin_1)
- U2 pad 55: Net-(J6-Pin_1) -> /MCU_Circuit/LEDWhite1
- U2 pad 56: unconnected-(U2-PD6-Pad56) -> /MCU_Circuit/LEDRed1
- U2 pad 57: unconnected-(U2-PB3-Pad57) -> /MCU_Circuit/LEDWhite2
- U2 pad 58: unconnected-(U2-PB4-Pad58) -> /MCU_Circuit/LEDRed2
- U2 pad 59: unconnected-(U2-PB5-Pad59) -> /MCU_Circuit/LEDWhite3
- U2 pad 60: unconnected-(U2-PB6-Pad60) -> /MCU_Circuit/LEDRed3
- U2 pad 61: unconnected-(U2-PB7-Pad61) -> /MCU_Circuit/LEDWhite4
- U2 pad 62: unconnected-(U2-PB8-Pad62) -> /MCU_Circuit/LEDRed4
Routing:
- net /MCU_Circuit/LEDRed4: track 0.00 -> 10.4 mm
- net /MCU_Circuit/LEDWhite1: track 0.00 -> 10.4 mm
- net /MCU_Circuit/LEDRed1: track 0.00 -> 9.51 mm
- net /MCU_Circuit/LEDWhite4: track 0.00 -> 9.41 mm
- net GND: track 25.6 -> 33.4 mm, vias 31 -> 53
- net /MCU_Circuit/LEDRed3: track 0.00 -> 7.15 mm
- net /MCU_Circuit/LEDWhite2: track 0.00 -> 6.80 mm
- net /MCU_Circuit/LEDWhite3: track 0.00 -> 6.69 mm
- net /MCU_Circuit/LEDRed2: track 0.00 -> 6.34 mm
- net /MCU_Circuit/NRST: track 47.7 -> 45.2 mm
- net Net-(D9-A): track 0.00 -> 1.20 mm
- net Net-(D8-A): track 0.00 -> 1.20 mm
- net Net-(D7-A): track 0.00 -> 1.20 mm
- net Net-(D6-A): track 0.00 -> 1.20 mm
- net Net-(D5-A): track 0.00 -> 1.20 mm
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Other:
- board text added: "CHG/ DCHG+"
- board text added: "CHG/ DCHG-"
- board text added: "CHK GND"
- board text added: "GND RDY SDA SCL FAULTNSFE FAULTN NSHIP WAKE 3V3"
- board text added: "GND RX TX MC0 TMS TCK NRST"
- board text added: "NRST GND"
- board text added: "SCL SDA WAKE GND"
